Commit message: Sensor Upgrade

File: src/my_robot/urdf/my_robot.xacro (robot description, xacro)
@@ -156,4 +156,6 @@
     </visual>
   </link>
+  <link name="camera_link_optical">
+  </link>
   <!--Joints-->
   <joint type="continuous" name="right_wheel_hinge">
@@ -185,3 +187,8 @@
     <axis xyz="0 1 0" rpy="0 0 0"/>
   </joint>
+  <joint name="camera_optical_joint" type="fixed">
+    <origin xyz="0 0 0" rpy="-1.5707 0 -1.5707"/>
+    <parent link="camera_link"/>
+    <child link="camera_link_optical"/>
+  </joint>
 </robot>

Commit message: remove the old existing camera and its shared object

File: src/my_robot/urdf/my_robot.xacro (robot description, xacro)
@@ -189,5 +189,5 @@
   <joint name="camera_optical_joint" type="fixed">
     <origin xyz="0 0 0" rpy="-1.5707 0 -1.5707"/>
-    <parent link="camera_link"/>
+    <parent link="camera"/>
     <child link="camera_link_optical"/>
   </joint>
